File: hardware/circuit/inki.kicad_pcb (KiCad board)
At the start: 2 copper layers, 47.2 x 55.5 mm, 47 parts, among them J1 connector epaper, J2 Conn_01x02_Socket, J3 Conn_01x02_Socket, J4 Conn_01x02_Socket, J5 Conn_01x02_Socket, J7 Conn_01x02_Socket, Q1 TSM260P02CX, Q2 MMBT3904, Q3 IRLML6344TRPBF, SW1 SW_DIP_x04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

Commit message: silk screen updates
Parts:
- renumbered C3 to 100n, 100n2 to 100n, 100n3 to 100n, 100n4 to 100n, 100n1 to 100n
Other:
- board text added: "100n"
- board text added: "10k"
- board text added: "1M"
- board text added: "1k"
- board text added: "200k"
- board text added: "22"
- board text added: "220"
- board text added: "2602"
- board text added: "3904"
- board text added: "4k7"
- board text added: "50k"
- board text added: "6344"
- board text added: "BAT54"
- board text added: "N4148"

Commit message: edit pcb: add bmp581
Parts:
- added U2: BMP581, Package_LGA:Bosch_LGA-8_2x2.5mm_P0.65mm_ClockwisePinNumbering, B.Cu at (47.0, 29.4)
- renumbered 100n to 100n1, 100n to 100n2, 100n to 100n3, 100n to 100n4, 100n to C3

Commit message: default config weathermap
Parts:
- added 100n5: C_Small, Capacitor_SMD:C_0805_2012Metric, B.Cu at (52.0, 38.5)
- U2: footprint Package_LGA:Bosch_LGA-8_2x2.5mm_P0.65mm_ClockwisePinNumbering -> inki:BMP581
- moved U2 13.0 mm to (52.0, 41.4)
Connections:
- U2 pad 1: unconnected-(U2-VDDIO-Pad1) -> Net-(J1-Pin_8)
- U2 pad 2: unconnected-(U2-SCK-Pad2) -> Net-(U1-SCL)
- U2 pad 3: unconnected-(U2-VSS-Pad3) -> GND
- U2 pad 4: unconnected-(U2-SDI/SDA/SDX-Pad4) -> Net-(U1-SDA)
- U2 pad 5: unconnected-(U2-SDO/ADDR-Pad5) -> Net-(J1-Pin_8)
- U2 pad 6: unconnected-(U2-CSB-Pad6) -> Net-(J1-Pin_8)
- U2 pad 7: unconnected-(U2-INT-Pad7) -> GND
- U2 pad 8: unconnected-(U2-VSS-Pad8) -> GND
Routing:
- net Net-(U1-SCL): track 22.5 -> 45.3 mm, vias 1 -> 2
- net Net-(J1-Pin_8): track 106.4 -> 127.8 mm, vias 1 -> 2
- net Net-(U1-SDA): track 22.4 -> 39.0 mm, vias 1 -> 3
- net GND: track 270.3 -> 275.3 mm, vias 5 -> 7
